File: kicad/openstint-preamp.kicad_sch (KiCad schematic)
At the start: 42 parts, among them J1 Phoenix PTS 1,5/ 2-5,0-H, J2 OUT, J3 Vin, J4 VNA_IN, J5 CAL_O, J6 CAL_S, J7 CAL_L, Q1 BFR106

Commit message: matching network, battery connection, oshw logo
Parts:
- removed L5: ?, Inductor_SMD:L_0603_1608Metric, symbol Device:L
- removed R12: 0, Resistor_SMD:R_0603_1608Metric, symbol Device:R
- added C13: 1500p, Capacitor_SMD:C_0603_1608Metric, symbol Device:C
- added C3: dnp, Capacitor_SMD:C_0603_1608Metric, symbol Device:C
- added R6, R7: 0, Resistor_SMD:R_0603_1608Metric, symbol Device:R
- added SYM1: Logo_Open_Hardware_Small, Symbol:OSHW-Logo2_9.8x8mm_SilkScreen, symbol Graphic:Logo_Open_Hardware_Small
- J3: footprint Connector_Wire:SolderWire-0.25sqmm_1x02_P4.2mm_D0.65mm_OD1.7mm -> Connector_JST:JST_PH_B2B-PH-K_1x02_P2.00mm_Vertical; LCSC (none) -> C131337
- L1: value 0 -> 820n; footprint Resistor_SMD:R_0603_1608Metric -> Inductor_SMD:L_0603_1608Metric; LCSC C21189 -> C18213078; now fitted
Connections:
- net GND: now also C13.2, C3.2; no longer L1.1
- net VCC: now also R6.2, R7.2; no longer C11.2, C12.2, C2.2, J3.1 (Pin_1), L6.2
- net loop_unbal: now also L1.1, C3.1; no longer L1.2
- net at C4.1: now also L1.2, C13.1
- new net +BATT: J3.1 (Pin_1), R6.1
- new net VBIAS: C11.2, C12.2, C2.2, L6.2, R7.1
Other:
- note added: "POWER SOURCE SELECTOR"
- note added: "To prevent damage of the radio, when external battery is used, move jumper from R7 to R6"
- moved on the sheet: C1, C10, C11, C12, C2, C4, C5, C6, C7, C8, C9, D1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
